Commit message: Minor changes and fixes

File: cocohrip_control/urdf/cocohrip_controlled.urdf.xacro (robot description, xacro)
@@ -28,5 +28,5 @@
     visual_parameters_file="$(arg visual_parameters_file)"
   >
-    <origin xyz="0 0 1" rpy="0 0 0" />
+    <origin xyz="0 0 0" rpy="0 0 0" />
   </xacro:cocohrip_cell>
   <!--Create the control tag for the UR robot-->
